File: hardware/common/RayCouplers.kicad_sch (KiCad schematic)
At the start: 54 parts, among them J1 RF OUT, J2 RF IN, J3 Conn_Coaxial, J4 Screw_Terminal_01x05, J5 Conn_Coaxial, T1 1:16T, T2 1:16T, U1 MCP6561U, U20 TLV3501AID, U21 MC74AC74DR2G

Commit message: RayCouplers: Finalize public engineering reference documentation
Parts:
- T1, T2: Sourcing_Status Owner-confirmed core identity, turns and wire; physical lea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 -> Established core identity, turns and wire; physical lead/po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
Changed lines of the file:
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@@
 			)
 		)
-		(property "Sourcing_Status" "Owner-confirmed core identity, turns and wire; physical lead/polarity mapping requires verification"
+		(property "Sourcing_Status" "Established core identity, turns and wire; physical lead/polarity mapping requires verification"
 			(at 106.68 74.93 0)
 			(effects
@@
 			)
 		)
-		(property "Sourcing_Status" "Owner-confirmed core identity, turns and wire; physical lead/polarity mapping requires verification"
+		(property "Sourcing_Status" "Established core identity, turns and wire; physical lead/polarity mapping requires verification"
 			(at 101.6 49.53 0)
 			(effects
