File: hardware/variants/2kw/RayCouplers.kicad_sch (KiCad schematic)
At the start: 54 parts, among them J1 RF OUT, J2 RF IN, J3 Conn_Coaxial, J4 Screw_Terminal_01x05, J5 Conn_Coaxial, T1 1:24T, T2 1:24T, U1 MCP6561U, U20 TLV3501AID, U21 MC74AC74DR2G

Commit message: RayCouplers: Finalize public engineering reference documentation
Parts:
- R1, R2, R3, R4, R5, R6: Sourcing_Status 100 ohm value approved; exact replacement MPN unresolved -> 100 ohm population value; exact replacement MPN unresolved
- T1, T2: Sourcing_Status Owner-confirmed core identity, turns and wire; physical lea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 -> Established core identity, turns and wire; physical lead/po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
Changed lines of the file:
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@@
 			)
 		)
-		(property "Sourcing_Status" "100 ohm value approved; exact replacement MPN unresolved"
+		(property "Sourcing_Status" "100 ohm population value; exact replacement MPN unresolved"
 			(at 64.77 74.93 0)
 			(effects
@@
 			)
 		)
-		(property "Sourcing_Status" "100 ohm value approved; exact replacement MPN unresolved"
+		(property "Sourcing_Status" "100 ohm population value; exact replacement MPN unresolved"
 			(at 76.2 80.01 0)
 			(effects
@@
 			)
 		)
-		(property "Sourcing_Status" "100 ohm value approved; exact replacement MPN unresolved"
+		(property "Sourcing_Status" "100 ohm population value; exact replacement MPN unresolved"
 			(at 137.16 80.01 0)
 			(effects
@@
 			)
 		)
-		(property "Sourcing_Status" "100 ohm value approved; exact replacement MPN unresolved"
+		(property "Sourcing_Status" "100 ohm population value; exact replacement MPN unresolved"
 			(at 64.77 85.09 0)
 			(effects
@@
 			)
 		)
-		(property "Sourcing_Status" "100 ohm value approved; exact replacement MPN unresolved"
+		(property "Sourcing_Status" "100 ohm population value; exact replacement MPN unresolved"
 			(at 148.59 74.93 0)
 			(effects
@@
 			)
 		)
-		(property "Sourcing_Status" "Owner-confirmed core identity, turns and wire; physical lead/polarity mapping requires verification"
+		(property "Sourcing_Status" "Established core identity, turns and wire; physical lead/polarity mapping requires verification"
 			(at 106.68 74.93 0)
 			(effects
@@
 			)
 		)
-		(property "Sourcing_Status" "100 ohm value approved; exact replacement MPN unresolved"
+		(property "Sourcing_Status" "100 ohm population value; exact replacement MPN unresolved"
 			(at 148.59 85.09 0)
 			(effects
@@
 			)
 		)
-		(property "Sourcing_Status" "Owner-confirmed core identity, turns and wire; physical lead/polarity mapping requires verification"
+		(property "Sourcing_Status" "Established core identity, turns and wire; physical lead/polarity mapping requires verification"
 			(at 101.6 49.53 0)
 			(effects
